Commit message: Update Lino physics for stability and multi-robot SLAM support

File: src/linorobot2/linorobot2_description/urdf/2wd_properties.urdf.xacro (robot description, xacro)
@@ -16,10 +16,10 @@
   <xacro:property name="wheel_torque" value="20" />
   <xacro:property name="front_caster_wheel" value="true" />
-  <xacro:property name="rear_caster_wheel" value="true" />
+  <xacro:property name="rear_caster_wheel" value="false" />
   <!-- set empty on the wheel_mesh_file to use geometry instead of mesh -->
   <xacro:property name="wheel_mesh_file" value="" />
   <!-- <xacro:property name="wheel_mesh_file" value="file://$(find linorobot2_description)/meshes/tire.dae" /> -->
   <xacro:property name="laser_pose">
-    <origin xyz="0.12 0 0.33" rpy="0 0 0"/>
+    <origin xyz="0.12 0 0.15" rpy="0 0 0"/>
   </xacro:property>
   <xacro:property name="depth_sensor_pose">

File: src/linorobot2/linorobot2_description/urdf/controllers/diff_drive.urdf.xacro (robot description, xacro)
@@ -5,8 +5,7 @@
         filename="gz-sim-diff-drive-system"
         name="gz::sim::systems::DiffDrive">
-        <topic>/cmd_vel</topic>
-        <!-- <frame_id>odom</frame_id> -->
-        <child_frame_id>base_footprint</child_frame_id>
-        <odom_topic>/odom/unfiltered</odom_topic>
+        <topic>/lino/cmd_vel</topic>
+        <frame_id>odom</frame_id>
+        <child_frame_id>lino/base_footprint</child_frame_id>
         <!-- <tf_topic>/tf</tf_topic> -->
         <left_joint>left_wheel_joint</left_joint>
@@ -20,5 +19,5 @@
       <plugin filename="gz-sim-joint-state-publisher-system"
         name="gz::sim::systems::JointStatePublisher">
-        <topic>/joint_states</topic>
+        <topic>joint_states</topic>
         <update_rate>50</update_rate>
         <joint_name>left_wheel_joint</joint_name>

File: src/linorobot2/linorobot2_description/urdf/mech/caster_wheel.urdf.xacro (robot description, xacro)
@@ -34,6 +34,12 @@
     </link>
     <gazebo reference="${side}_caster_wheel_link">
-        <mu1>0.01</mu1>
-        <mu2>0.01</mu2>
+      <surface>
+        <friction>
+          <ode>
+            <mu>0.001</mu>
+            <mu2>0.001</mu2>
+          </ode>
+        </friction>
+      </surface>
     </gazebo>
     <joint name="${side}_caster_wheel_joint" type="fixed">

File: src/linorobot2/linorobot2_description/urdf/sensors/depth_sensor.urdf.xacro (robot description, xacro)
@@ -42,4 +42,7 @@
       <xacro:insert_block name="origin" />
     </joint>
+    <gazebo reference="camera_to_base_link">
+      <disableFixedJointLumping>true</disableFixedJointLumping>
+    </gazebo>
     <link name="camera_depth_link"/>
     <joint name="camera_depth_joint" type="fixed">
@@ -48,4 +51,7 @@
       <child link="camera_depth_link"/>
     </joint>
+    <gazebo reference="camera_depth_joint">
+      <disableFixedJointLumping>true</disableFixedJointLumping>
+    </gazebo>
     <link name="camera_depth_optical_frame"/>
     <joint name="camera_depth_optical_joint" type="fixed">
@@ -54,12 +60,15 @@
       <child link="camera_depth_optical_frame"/>
     </joint>
+    <gazebo reference="camera_depth_optical_joint">
+      <disableFixedJointLumping>true</disableFixedJointLumping>
+    </gazebo>
     <gazebo reference="camera_link">
       <sensor name="camera" type="rgbd_camera">
-        <topic>/camera</topic>
+        <topic>/lino/camera</topic>
         <update_rate>30.0</update_rate>
         <always_on>true</always_on>
         <visualize>true</visualize>
         <camera>
-          <optical_frame_id>camera_depth_optical_frame</optical_frame_id>
+          <optical_frame_id>lino/camera_depth_optical_frame</optical_frame_id>
           <horizontal_fov>1.50098</horizontal_fov>
           <image>

File: src/linorobot2/linorobot2_description/urdf/sensors/generic_laser.urdf.xacro (robot description, xacro)
@@ -11,5 +11,5 @@
       max_range="12.0"
       frame_id="laser"
-      topic_name="/scan"
+      topic_name="scan"
     >
       <xacro:insert_block name="origin" />
@@ -25,5 +25,5 @@
       max_range="5.5"
       frame_id="base_laser"
-      topic_name="/base/scan"
+      topic_name="base_scan"
     >
       <xacro:insert_block name="origin" />

File: src/linorobot2/linorobot2_description/urdf/sensors/imu.urdf.xacro (robot description, xacro)
@@ -13,5 +13,5 @@
     <gazebo reference="imu_link">
       <sensor name="imu_sensor" type="imu">
-        <topic>/imu/data</topic>
+        <topic>imu/data</topic>
         <update_rate>50</update_rate>
         <always_on>true</always_on>

File: src/linorobot2/linorobot2_description/urdf/sensors/laser.urdf.xacro (robot description, xacro)
@@ -41,8 +41,11 @@
       <xacro:insert_block name="origin" />
     </joint>
+    <gazebo reference="${frame_id}_to_base_link">
+      <disableFixedJointLumping>true</disableFixedJointLumping>
+    </gazebo>
     <gazebo reference="${frame_id}">
       <sensor name="gpu_lidar" type="gpu_lidar">
-        <topic>${topic_name}</topic>
-        <gz_frame_id>${frame_id}</gz_frame_id>
+        <topic>/lino/${topic_name}</topic>
+        <gz_frame_id>lino/${frame_id}</gz_frame_id>
         <update_rate>${update_rate}</update_rate>
         <always_on>true</always_on>

File: src/linorobot2/linorobot2_description/urdf/sensors/plugins.urdf.xacro (robot description, xacro)
@@ -1,3 +1,4 @@
 <robot xmlns:xacro="http://ros.org/wiki/xacro">
+  <!--
   <gazebo>
     <plugin
@@ -7,3 +8,4 @@
     </plugin>
   </gazebo>
+  -->
 </robot>
